File: semtech-dev-board.brd (EAGLE design)
At the start: 100 x 80 mm, 21 parts, among them Q1 OPTIONAL, Q2 BSS123, Q3 BSS84, U1 MIC5219 3.3V, X1 BU-SMA-G, X2 BU-SMA-G, X3 BU-SMA-G, X4 BU-SMA-G, X5 BU-SMA-G

Commit message: adjustments based on Friday meeting
Parts:
- added C10, C9: 6pF, rcl:C0805
- added C3, C4, C5, C6, C7, C8: 100nF, rcl:C0805
- added R3, R5, R6, R7: 0, rcl:R0805
- added R4: (no value), rcl:R0805
- added R8: 1k, rcl:R0805
- added TP1, TP2, TP3, TP4, TP5, TP6: TEST-POINT, low-gain-radio:2MM-TEST-POINT
- JP1: device pinhead:2X03 -> pinhead:1X04
- Q1: value OPTIONAL -> (none)
- moved JP1 79.9 mm to (-4.57, -3.81), turned to 0 degrees
- moved C2 39.0 mm to (24.4, 37.8), turned to 270 degrees
- moved C1 27.5 mm to (17.0, 45.2)
- moved U1 27.2 mm to (23.1, 44.7), turned to 180 degrees
- moved JP2 25.9 mm to (39.4, 2.54)
- moved U$2 23.6 mm to (27.7, 65.8), turned to 180 degrees
- moved X2 20.1 mm to (64.0, 28.2)
- moved X4 18.3 mm to (64.0, 40.1)
- moved U$1 15.3 mm to (29.2, 22.9)
- moved JP3 13.0 mm to (18.0, 63.2), turned to 270 degrees
- moved R2 11.7 mm to (49.5, 40.6), turned to 270 degrees
- moved Q2 10.9 mm to (39.4, 35.6), turned to 90 degrees
- moved X5 9.94 mm to (5.59, 43.4)
- moved X1 9.67 mm to (5.84, 20.8)
- moved X3 9.18 mm to (5.59, 32.8)
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Connections:
- net N$10 renamed DIO2
- net N$11 renamed DIO3
- net N$12 renamed DIO4
- net N$13 renamed DIO5
- net N$14 renamed RFI_HF
- net N$15 renamed RFI_LF
- net N$16 renamed RFO_HF
- net N$17 renamed RFO_LF
- net N$19 renamed BP
- net N$21 renamed PA_BOOST
- net N$3 renamed SPI_SCK
- net N$8 renamed DIO0
- net N$9 renamed DIO1
- removed net N$18: JP3.2, U$2.1, U1.1, U1.3
- removed net N$22: Q1.1, U$1.5
- removed net N$23: Q1.2, U$1.6
- removed net N$24: Q2.1, Q3.1, U$1.20
- removed net N$25: S1.A1, U$1.7
- removed net N$5: JP1.4, U$1.18
- new net 5219_EN: R4.1, TP1.1, U1.3
- new net AGND: C3.2, C4.2, C5.2, R5.2, R6.2, U$1.0, U$1.15, U$1.23, U$1.26, X1.2, X1.3, X1.4, X1.5, X2.2, X2.3, X2.4, X2.5, X3.2, X3.3, X3.4, X3.5, X4.2, X4.3, X4.4, X4.5, X5.2, X5.3, X5.4, X5.5
- new net N$4: R8.1, S1.A
- new net RXTX: Q2.1, Q3.1, TP3.1, U$1.20
- new net SPI_MOSI: JP1.2, U$1.18
- new net SPI_NSS: JP1.4, U$1.19
- new net SX1236_RST: S1.A1, TP4.1, U$1.7
- new net VBAT: C6.1, C7.1, C8.1, R7.1, U$1.3
- new net VREG_IN: R3.2, R4.2, TP6.1, U1.1
- new net VR_ANA: C5.1, U$1.2
- new net VR_DIG: C4.1, U$1.4
- new net VR_PA: C3.1, U$1.25
- new net V_IN: JP3.2, R3.1, TP2.1, U$2.1
- new net XTALB: C9.1, Q1.1, U$1.6
- net +3V3: now also R7.2, R8.2, TP5.1, U$1.14, U$1.24; no longer JP1.2, S1.A
- net GND: now also C10.2, C6.2, C7.2, C8.2, C9.2, R5.1, R6.1; no longer JP1.6, U$1.0, U$1.15, U$1.23, U$1.26, X1.2, X1.3, X1.4, X1.5, X2.2, X2.3, X2.4, X2.5, X3.2, X3.3, X3.4, X3.5, X4.2, X4.3, X4.4, X4.5, X5.2, X5.3, X5.4, X5.5
- net N$2: now also C10.1, Q1.2, U$1.5; no longer JP1.5, U$1.19
Routing:
- net N$4: track 0.00 -> 41.6 mm
- net N$2: track 0.00 -> 36.6 mm
- net RFO_HF: track 0.00 -> 34.4 mm
- net +3V3: track 0.00 -> 34.2 mm, vias 0 -> 1
- net PA_BOOST: track 0.00 -> 32.9 mm
- net RFI_LF: track 0.00 -> 31.8 mm
- net RFI_HF: track 0.00 -> 29.8 mm
- net XTALB: track 0.00 -> 28.6 mm
- net RFO_LF: track 0.00 -> 26.3 mm
- net DIO5: track 0.00 -> 25.6 mm
- net DIO4: track 0.00 -> 24.9 mm
- net DIO3: track 0.00 -> 24.0 mm
- net DIO2: track 0.00 -> 23.4 mm
- net DIO1: track 0.00 -> 22.6 mm
- net DIO0: track 0.00 -> 21.7 mm
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- added copper zone on layer 16, net AGND
Other:
- board size 100 x 80 mm -> 69.5 x 80 mm

Commit message: Updates from Sunday meeting
Parts:
- removed X5: BU-SMA-G, con-coax:BU-SMA-G
- added TP7: TEST-POINT, low-gain-radio:2MM-TEST-POINT
- JP2: device pinhead:1X06 -> pinhead:1X07
- moved JP1 61.0 mm to (56.1, 2.54)
- moved R8 38.2 mm to (14.0, 22.1), turned to 90 degrees
- moved R7 1.55 mm to (13.2, 34.8), turned to 180 degrees
Connections:
- removed net DIO0: JP2.1, U$1.8
- removed net DIO1: JP2.2, U$1.9
- removed net DIO2: JP2.3, U$1.10
- removed net DIO3: JP2.4, U$1.11
- removed net DIO4: JP2.5, U$1.12
- removed net DIO5: JP2.6, U$1.13
- new net N$10: JP2.4, U$1.10
- new net N$11: JP2.5, U$1.11
- new net N$12: JP2.6, U$1.12
- new net N$13: JP2.7, U$1.13
- new net N$5: JP2.2, U$1.8
- new net N$9: JP2.3, U$1.9
- net AGND: no longer X5.2, X5.3, X5.4, X5.5
- net PA_BOOST: now also TP7.1; no longer X5.1
- net RXTX: now also JP2.1
Routing:
- net N$4: track 41.6 -> 0.00 mm
- net DIO5: track 25.6 -> 0.00 mm
- net DIO4: track 24.9 -> 0.00 mm
- net DIO3: track 24.0 -> 0.00 mm
- net DIO2: track 23.4 -> 0.00 mm
- net DIO1: track 22.6 -> 0.00 mm
- net DIO0: track 21.7 -> 0.00 mm
- net PA_BOOST: track 32.9 -> 26.0 mm

Commit message: added biasing circuitry to match ref design for sx1233
Parts:
- removed R5, R6: 0, rcl:R0805
- added C11, C12, C13, C14, C15, C16, C17, C18, C19, C20, C21, C22, C23: 100nF, rcl:C0805
- added L1, L2, L3, L4, L5, L6, L7, L8: (no value), rcl:L3230M
- moved C3 61.3 mm to (-11.7, -11.9), turned to 0 degrees
Connections:
- removed net RFO_LF: U$1.28, X3.1
- removed net VR_PA: C3.1, U$1.25
- new net N$14: C5.1, U$1.2
- new net N$15: C23.1, C3.1, L2.1, L8.1, U$1.25
- new net N$16: L1.1, U$1.28
- new net N$17: C11.1, C12.1, L1.2, L2.2
- new net N$18: L7.2, U$1.22
- new net N$19: C17.1, C18.1, L7.1, L8.2
- new net N$22: C18.2, C19.1, L5.2
- new net N$23: C19.2, C20.1, C21.1, L5.1, L6.2
- new net N$26: C12.2, C13.1, L3.2
- new net N$27: C13.2, C14.1, L3.1, L4.2
- new net N$28: C14.2, C16.1, L4.1
- net +3V3: no longer U$1.14, U$1.24
- net AGND: now also C11.2, C15.2, C16.2, C17.2, C21.2, C22.2, C23.2; no longer R5.2, R6.2
- net GND: no longer R5.1, R6.1
- net RFO_HF: now also C20.2, C22.1, L6.1; no longer U$1.22
- net VBAT: now also U$1.14, U$1.24
- net VR_ANA: now also U$1.4; no longer C5.1, U$1.2
- net VR_DIG: no longer U$1.4
Routing:
- net RFO_LF: track 26.3 -> 0.00 mm
- net VBAT: track 8.11 -> 0.00 mm
- net VR_ANA: track 6.02 -> 0.00 mm
- net AGND: track 18.5 -> 12.9 mm
- net SX1236_RST: track 20.6 -> 15.8 mm
- net RXTX: track 17.4 -> 12.6 mm
- net +3V3: track 34.2 -> 30.2 mm
- net VR_PA: track 3.44 -> 0.00 mm
- net VR_DIG: track 8.51 -> 6.40 mm
- net RFO_HF: track 34.4 -> 33.7 mm

Commit message: formatted sch
Parts:
- added JP4: (no value), pinhead:1X04
Connections:
- net N$16 renamed RFO_LF
- removed net N$18: L7.2, U$1.22
- new net N$24: C3.1, JP4.1, L2.2
- new net VR_PA: JP4.2, JP4.3, U$1.25
- net GND: now also JP3.2; no longer JP3.1
- net N$15: now also JP4.4, L8.2; no longer C3.1, L2.1, L8.1, U$1.25
- net N$17: now also L2.1; no longer L2.2
- net N$19: now also L8.1; no longer L8.2
- net N$27: now also C15.1
- net N$28: now also X3.1
- net RFO_HF: now also L7.2, U$1.22
- net V_IN: now also JP3.1; no longer JP3.2
Changed lines of the file:
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@@
 <element name="L8" library="rcl" package="L3230M" value="" x="-11.176" y="-118.618"/>
 <element name="C23" library="rcl" package="C0805" value="100nF" x="-11.684" y="-125.476"/>
+<element name="JP4" library="pinhead" package="1X04" value="" x="-2.286" y="-136.144"/>
 </elements>
 <signals>
@@
 <contactref element="U$2" pad="GND2"/>
 <contactref element="U$2" pad="5"/>
-<contactref element="JP3" pad="1"/>
 <contactref element="U1" pad="2"/>
 <contactref element="C2" pad="2"/>
@@
 <contactref element="C7" pad="2"/>
 <contactref element="C6" pad="2"/>
+<contactref element="JP3" pad="2"/>
 <wire x1="26.386" y1="61.261" x2="31.411" y2="64.086" width="0" layer="19" extent="1-1"/>
 <wire x1="23.961" y1="64.086" x2="26.386" y2="61.261" width="0" layer="19" extent="1-1"/>
-<wire x1="18.034" y1="64.516" x2="23.961" y2="64.086" width="0" layer="19" extent="1-1"/>
+<wire x1="18.034" y1="61.976" x2="23.961" y2="64.086" width="0" layer="19" extent="1-1"/>
 <wire x1="23.114" y1="46.0041" x2="26.386" y2="61.261" width="0" layer="19" extent="1-1"/>
 <wire x1="17.968" y1="45.212" x2="23.114" y2="46.0041" width="0" layer="19" extent="1-1"/>
@@
 <contactref element="C22" pad="1"/>
 <contactref element="C20" pad="2"/>
+<contactref element="U$1" pad="22"/>
+<contactref element="L7" pad="2"/>
+<wire x1="-12.634" y1="-104.394" x2="-9.776" y2="-111.252" width="0" layer="19" extent="1-1"/>
 <wire x1="-10.734" y1="-98.298" x2="-12.634" y2="-104.394" width="0" layer="19" extent="1-1"/>
 <wire x1="-7.496" y1="-85.344" x2="-10.734" y2="-98.298" width="0" layer="19" extent="1-1"/>
-<wire x1="34.51" y1="29.938" x2="-7.496" y2="-85.344" width="0" layer="19" extent="1-1"/>
+<wire x1="34.51" y1="29.185" x2="-7.496" y2="-85.344" width="0" layer="19" extent="1-1"/>
+<wire x1="34.51" y1="29.938" x2="34.51" y2="29.185" width="0" layer="19" extent="1-1"/>
 </signal>
 <signal name="XTALB">
@@
 <signal name="V_IN">
 <contactref element="U$2" pad="1"/>
-<contactref element="JP3" pad="2"/>
 <contactref element="R3" pad="1"/>
 <contactref element="TP2" pad="1"/>
+<contactref element="JP3" pad="1"/>
 <wire x1="24.892" y1="56.576" x2="28.986" y2="61.261" width="0" layer="19" extent="1-1"/>
 <wire x1="19.05" y1="53.848" x2="24.892" y2="56.576" width="0" layer="19" extent="1-1"/>
-<wire x1="18.034" y1="61.976" x2="19.05" y2="53.848" width="0" layer="19" extent="1-1"/>
+<wire x1="18.034" y1="64.516" x2="24.892" y2="56.576" width="0" layer="19" extent="1-1"/>
 </signal>
 <signal name="PA_BOOST">
@@
 </signal>
 <signal name="N$15">
-<contactref element="U$1" pad="25"/>
-<contactref element="L2" pad="1"/>
-<contactref element="L8" pad="1"/>
 <contactref element="C23" pad="1"/>
-<contactref element="C3" pad="1"/>
-<wire x1="-12.576" y1="-118.618" x2="-12.634" y2="-125.476" width="0" layer="19" extent="1-1"/>
-<wire x1="-12.576" y1="-26.162" x2="-12.576" y2="-118.618" width="0" layer="19" extent="1-1"/>
-<wire x1="-12.634" y1="-11.938" x2="-12.576" y2="-26.162" width="0" layer="19" extent="1-1"/>
-<wire x1="32.56" y1="29.185" x2="-12.634" y2="-11.938" width="0" layer="19" extent="1-1"/>
-</signal>
-<signal name="N$16">
+<contactref element="L8" pad="2"/>
+<contactref element="JP4" pad="4"/>
+<wire x1="-9.776" y1="-118.618" x2="-12.634" y2="-125.476" width="0" layer="19" extent="1-1"/>
+<wire x1="1.524" y1="-136.144" x2="-12.634" y2="-125.476" width="0" layer="19" extent="1-1"/>
+</signal>
+<signal name="RFO_LF">
 <contactref element="U$1" pad="28"/>
 <contactref element="L1" pad="1"/>
@@
 <signal name="N$17">
 <contactref element="L1" pad="2"/>
-<contactref element="L2" pad="2"/>
 <contactref element="C11" pad="1"/>
 <contactref element="C12" pad="1"/>
+<contactref element="L2" pad="1"/>
 <wire x1="-12.634" y1="-33.02" x2="-12.634" y2="-39.116" width="0" layer="19" extent="1-1"/>
-<wire x1="-9.776" y1="-26.162" x2="-12.634" y2="-33.02" width="0" layer="19" extent="1-1"/>
-<wire x1="-9.776" y1="-18.796" x2="-9.776" y2="-26.162" width="0" layer="19" extent="1-1"/>
+<wire x1="-12.576" y1="-26.162" x2="-12.634" y2="-33.02" width="0" layer="19" extent="1-1"/>
+<wire x1="-9.776" y1="-18.796" x2="-12.576" y2="-26.162" width="0" layer="19" extent="1-1"/>
 </signal>
 <signal name="N$19">
-<contactref element="C17" pad="1"/>
 <contactref element="C18" pad="1"/>
 <contactref element="L7" pad="1"/>
-<contactref element="L8" pad="2"/>
-<wire x1="-12.576" y1="-111.252" x2="-9.776" y2="-118.618" width="0" layer="19" extent="1-1"/>
+<contactref element="L8" pad="1"/>
+<contactref element="C17" pad="1"/>
+<wire x1="-12.576" y1="-111.252" x2="-12.576" y2="-118.618" width="0" layer="19" extent="1-1"/>
 <wire x1="-12.634" y1="-92.202" x2="-12.576" y2="-111.252" width="0" layer="19" extent="1-1"/>
 <wire x1="-2.474" y1="-84.582" x2="-12.634" y2="-92.202" width="0" layer="19" extent="1-1"/>
-</signal>
-<signal name="N$18">
-<contactref element="U$1" pad="22"/>
-<contactref element="L7" pad="2"/>
-<wire x1="34.51" y1="29.185" x2="-9.776" y2="-111.252" width="0" layer="19" extent="1-1"/>
 </signal>
 <signal name="N$22">
@@
 <contactref element="C14" pad="1"/>
 <contactref element="C13" pad="2"/>
+<contactref element="C15" pad="1"/>
+<wire x1="-12.634" y1="-66.294" x2="-12.634" y2="-72.39" width="0" layer="19" extent="1-1"/>
 <wire x1="-10.734" y1="-60.198" x2="-12.634" y2="-66.294" width="0" layer="19" extent="1-1"/>
 <wire x1="-9.776" y1="-53.34" x2="-10.734" y2="-60.198" width="0" layer="19" extent="1-1"/>
@@
 <contactref element="C16" pad="1"/>
 <contactref element="C14" pad="2"/>
+<contactref element="X3" pad="1"/>
 <wire x1="-10.734" y1="-66.294" x2="-12.634" y2="-78.486" width="0" layer="19" extent="1-1"/>
 <wire x1="-12.576" y1="-53.34" x2="-10.734" y2="-66.294" width="0" layer="19" extent="1-1"/>
+<wire x1="5.588" y1="32.766" x2="-12.576" y2="-53.34" width="0" layer="19" extent="1-1"/>
+</signal>
+<signal name="N$24">
+<contactref element="C3" pad="1"/>
+<contactref element="L2" pad="2"/>
+<contactref element="JP4" pad="1"/>
+<wire x1="-9.776" y1="-26.162" x2="-6.096" y2="-136.144" width="0" layer="19" extent="1-1"/>
+<wire x1="-12.634" y1="-11.938" x2="-9.776" y2="-26.162" width="0" layer="19" extent="1-1"/>
+</signal>
+<signal name="VR_PA">
+<contactref element="U$1" pad="25"/>
+<contactref element="JP4" pad="2"/>
+<contactref element="JP4" pad="3"/>
+<wire x1="-1.016" y1="-136.144" x2="-3.556" y2="-136.144" width="0" layer="19" extent="1-1"/>
+<wire x1="32.56" y1="29.185" x2="-1.016" y2="-136.144" width="0" layer="19" extent="1-1"/>
 </signal>
 </signals>

Commit message: started 4 layer board
Parts:
- removed LED2: (no value), led:CHIP-LED0805
- removed Q3: BSS84, transistor-small-signal:SOT23
- removed R7: 0, rcl:R0805
- removed R8: 1k, rcl:R0805
- removed TP3: TEST-POINT, low-gain-radio:2MM-TEST-POINT
- removed U$1: SEMTECH_SX1236, low-gain-radio:QFN28
- removed U$2: MICRO-USB, microusb:MICRO-USB
- added JP5: (no value), pinhead:1X02
- added R5: (no value), rcl:R0805
- added U2: (no value), microusb:USB-MICRO-SMD
- added U3: MIC5219 3.3V, SparkFun-IC-Power:SOT23-5
- C1: value 470pF -> 100nF
- C10, C9: value 6pF -> 100nF
- C2: value 1uF -> 100nF
- C21: value 100nF -> 470pF
- C23: value 100nF -> 1uF
- C6, C7: value 100nF -> 6pF
- JP1: device pinhead:1X04 -> pinhead:1X07
- JP2: device pinhead:1X07 -> pinhead:1X04
- L5: device rcl:L3230M -> rcl:L1812
- Q1: value (none) -> BSS123; device crystal:SM49 -> transistor-small-signal:SOT23
- Q2: value BSS123 -> (none); device transistor-small-signal:SOT23 -> crystal:SM49
- R2: value (none) -> 1k; device rcl:M0805 -> rcl:R0805
- R4: value (none) -> 0
- U1: value MIC5219 3.3V -> SEMTECH_SX1236; device SparkFun-IC-Power:SOT23-5 -> low-gain-radio:QFN28
- moved L7 235.1 mm to (137.2, 71.1), turned to 180 degrees
- moved C20 231.5 mm to (144.8, 72.4), turned to 90 degrees
- moved L8 228.8 mm to (139.7, 53.3), turned to 180 degrees
- moved C22 222.2 mm to (146.1, 52.1), turned to 270 degrees
- moved C17 212.3 mm to (137.2, 76.2)
- moved C19 209.1 mm to (139.7, 58.4)
- moved L5 204.8 mm to (119.4, 72.4), turned to 90 degrees
- moved C16 203.9 mm to (129.5, 68.6), turned to 90 degrees
- moved C18 203.7 mm to (132.1, 52.1), turned to 270 degrees
- moved C14 199.7 mm to (128.3, 76.2)
- moved JP4 197.8 mm to (58.4, 52.1)
- moved C23 194.5 mm to (14.0, 67.3)
- moved L6 189.6 mm to (123.2, 53.3)
- moved C15 187.9 mm to (123.2, 58.4), turned to 180 degrees
- moved C13 170.5 mm to (115.6, 53.3)
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Connections:
- removed net N$20: LED2.C, Q3.2
- removed net N$7: LED2.A, R2.1
- new net RFO_HF_OUT: C19.2, C22.1, L8.1, X3.1
- net +3V3: now also C23.1, R3.2, U3.5; no longer C2.1, R7.2, R8.2, U1.5
- net 5219_EN: now also R5.1, U3.3; no longer R4.1, U1.3
- net AGND: now also C10.2, C12.2, C18.2, C20.2, C8.2, C9.2, U1.0, U1.15, U1.23, U1.26; no longer C11.2, C15.2, C17.2, C21.2, C23.2, C3.2, U$1.0, U$1.15, U$1.23, U$1.26
- net BP: now also C21.1, U3.4; no longer C1.1, U1.4
- net GND: now also C21.2, C23.2, C3.2, JP5.2, Q1.2, U2.GND1, U3.2; no longer C10.2, C8.2, C9.2, Q2.2, Q3.3, U$2.5, U$2.GND1, U$2.GND2, U1.2
- net N$1: now also Q1.3; no longer Q2.3
- net N$10: now also JP1.4, U1.10; no longer JP2.4, U$1.10
- net N$11: now also JP1.5, U1.11; no longer JP2.5, U$1.11
- net N$12: now also JP1.6, U1.12; no longer JP2.6, U$1.12
- net N$13: now also JP1.7, U1.13; no longer JP2.7, U$1.13
- net N$14: now also C4.1, U1.2; no longer C5.1, U$1.2
- net N$15: now also C9.1, L2.2; no longer C23.1, L8.2
- net N$17: now also C10.1, L1.1, L3.2; no longer C12.1, L1.2, L2.1
- net N$19: now also C12.1, C13.1, L2.1, L4.1; no longer C17.1, C18.1, L7.1, L8.1
- net N$2: now also C7.1, Q2.2, U1.5; no longer C10.1, Q1.2, U$1.5
- net N$22: now also C13.2, C15.1, L6.2; no longer C18.2, C19.1, L5.2
- net N$23: now also C15.2, C18.1, C19.1, L6.1, L8.2; no longer C19.2, C20.1, C21.1, L5.1, L6.2
- net N$24: now also C8.1, L1.2; no longer C3.1, L2.2
- net N$26: now also C11.2, C14.1, L5.2; no longer C12.2, C13.1, L3.2
- net N$27: now also C14.2, C16.1, C17.1, L5.1, L7.2; no longer C13.2, C14.1, C15.1, L3.1, L4.2
- net N$28: now also C17.2, C20.1, L7.1, X2.1; no longer C14.2, C16.1, L4.1, X3.1
- net N$3: now also JP2.1, U1.17; no longer JP1.1, U$1.17
- net N$4: now also R2.1; no longer R8.1
- net N$5: now also JP1.2, U1.8; no longer JP2.2, U$1.8
- net N$9: now also JP1.3, U1.9; no longer JP2.3, U$1.9
- net PA_BOOST: now also U1.27; no longer U$1.27
- net RFI_HF: now also U1.21, X4.1; no longer U$1.21, X2.1
- net RFI_LF: now also U1.1; no longer U$1.1
- net RFO_HF: now also L4.2, U1.22; no longer C20.2, C22.1, L6.1, L7.2, U$1.22, X4.1
- net RFO_LF: now also L3.1, U1.28; no longer L1.1, U$1.28
- net RXTX: now also JP1.1, JP3.1, Q1.1, U1.20; no longer JP2.1, Q2.1, Q3.1, TP3.1, U$1.20
- net SPI_MOSI: now also JP2.2, U1.18; no longer JP1.2, U$1.18
- net SPI_NSS: now also JP2.4, U1.19; no longer JP1.4, U$1.19
- net SPI_SCK: now also JP2.3, U1.16; no longer JP1.3, U$1.16
- net SX1236_RST: now also U1.7; no longer U$1.7
- net VBAT: now also C1.1, C2.1, C3.1, R3.1, U1.14, U1.24, U1.3; no longer C6.1, C7.1, C8.1, R7.1, U$1.14, U$1.24, U$1.3
- net VREG_IN: now also R5.2, U3.1; no longer R3.2, U1.1
- net VR_ANA: now also U1.4; no longer U$1.4
- net VR_DIG: now also C5.1; no longer C4.1
- net VR_PA: now also U1.25; no longer U$1.25
- net V_IN: now also JP5.1, R4.1, U2.VBUS1; no longer JP3.1, R3.1, U$2.1
- net XTALB: now also C6.1, Q2.1, U1.6; no longer C9.1, Q1.1, U$1.6
Routing:
- net AGND: track 12.9 -> 72.4 mm, vias 2 -> 0
- net N$2: track 36.6 -> 0.00 mm
- net RFO_HF: track 33.7 -> 0.00 mm
- net RFI_LF: track 31.8 -> 0.00 mm
- net +3V3: track 30.2 -> 0.00 mm, vias 1 -> 0
- net RFI_HF: track 29.8 -> 0.00 mm
- net XTALB: track 28.6 -> 0.00 mm
- net PA_BOOST: track 26.0 -> 0.00 mm
- net SPI_NSS: track 21.4 -> 0.00 mm
- net SX1236_RST: track 15.8 -> 0.00 mm
- net RXTX: track 12.6 -> 0.00 mm, vias 2 -> 0
- net N$20: track 6.84 -> 0.00 mm
- net VR_DIG: track 6.40 -> 0.00 mm
- net N$1: track 5.46 -> 0.00 mm
- added copper zone on layer 2, net AGND
- removed copper zone on layer 16, net AGND
- removed copper zone on layer 1, net GND
Other:
- board size 69.5 x 80 mm -> 160 x 100 mm

Commit message: Fixed inductors
Parts:
- moved C5 36.4 mm to (40.6, 35.6), turned to 180 degrees
- moved LED1 32.3 mm to (5.84, 38.4)
- moved R1 31.5 mm to (10.9, 41.4), turned to 0 degrees
- moved S1 26.0 mm to (40.4, -3.05)
- moved C4 25.5 mm to (44.5, 41.9), turned to 90 degrees
- moved R2 25.4 mm to (49.5, 3.81)
- moved TP4 25.0 mm to (59.7, 2.54)
- moved C6 24.2 mm to (42.7, 30.0)
- moved Q1 22.6 mm to (12.4, 36.8)
- moved C1 17.2 mm to (55.0, 30.7), turned to 270 degrees
- moved JP3 14.0 mm to (2.54, 36.8)
- moved U2 12.7 mm to (1.27, 54.6)
- moved C2 12.0 mm to (52.1, 43.2), turned to 90 degrees
- moved JP5 11.5 mm to (2.54, 45.7)
- moved Q2 8.82 mm to (32.5, 31.5), turned to 180 degrees
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Connections:
- net N$10 renamed DIO2
- net N$11 renamed DIO3
- net N$12 renamed DIO4
- net N$13 renamed DIO5
- net N$17 renamed RFO_LF_PA
- net N$19 renamed RFO_HF_PA
- net N$22 renamed RFO_HF_1
- net N$23 renamed RFO_HF_2
- net N$26 renamed RFO_LF_1
- net N$27 renamed RFO_LF_2
- net N$28 renamed RFO_LF_OUT
- net N$4 renamed RST_SUP
- net N$5 renamed DIO0
- net N$9 renamed DIO1
- removed net N$14: C4.1, U1.2
- removed net SPI_MOSI: JP2.2, U1.18
- removed net SPI_SCK: JP2.3, U1.16
- new net N$4: JP2.2, U1.17
- new net N$5: JP2.1, U1.16
- net N$3: now also JP2.3, U1.18; no longer JP2.1, U1.17
- net VR_ANA: now also C4.1, U1.2; no longer U1.4
- net VR_DIG: now also U1.4
Routing:
- net SPI_NSS: track 0.00 -> 81.2 mm
- net DIO5: track 0.00 -> 61.6 mm
- net DIO4: track 0.00 -> 59.5 mm
- net DIO3: track 0.00 -> 57.2 mm
- net DIO2: track 0.00 -> 55.1 mm
- net DIO1: track 0.00 -> 53.1 mm
- net DIO0: track 0.00 -> 50.3 mm
